File: Hardware/BEEP_0.1/PCA9548A.sch (EAGLE design)
At the start: 13 parts, among them IC1 PCA9548A

Commit message: Add branding ;) enhance PCBs finish Easy RGB Board add Texas Instruments libray from Element 14 add dxf import ulp for eagle add Script for easy eagle export to pdf for etching minor cleanup
Parts:
- added U$1: LOGO-COPPER4, Branding:LOGO-COPPER4
Other:
- moved on the sheet: A01, A2, C1, I2C, IC1, JP3, JP4, POWER, R1, R2, R3, R4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
