File: Hardware/BEEP_0.1/ATMEGA168.sch (EAGLE design)
At the start: 19 parts, among them IC1 ATMEGA48/88/168-AU, Q1 20Mhz

Commit message: Add branding ;) enhance PCBs finish Easy RGB Board add Texas Instruments libray from Element 14 add dxf import ulp for eagle add Script for easy eagle export to pdf for etching minor cleanup
Parts:
- added U$1: LOGO-COPPER4, Branding:LOGO-COPPER4
Other:
- moved on the sheet: C1, C2, C3, C4, C5, IC1, ISP, JP2, JP3, JP4, JP5, POWER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

Commit message: rotate reset button on atmega board remove GND under TCS3103
Connections:
- net GND: now also S1.P; no longer S1.S1
- net RST: now also S1.S1; no longer S1.P
Changed lines of the file:
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@@
 <wire x1="25.4" y1="99.06" x2="20.32" y2="99.06" width="0.1524" layer="91"/>
 <wire x1="20.32" y1="99.06" x2="20.32" y2="104.14" width="0.1524" layer="91"/>
-<pinref part="S1" gate="1" pin="S1"/>
-<wire x1="25.4" y1="99.06" x2="30.48" y2="99.06" width="0.1524" layer="91"/>
-<wire x1="30.48" y1="99.06" x2="30.48" y2="104.14" width="0.1524" layer="91"/>
-<junction x="25.4" y="99.06"/>
+<pinref part="S1" gate="1" pin="P"/>
+<wire x1="20.32" y1="104.14" x2="20.32" y2="106.68" width="0.1524" layer="91"/>
+<junction x="20.32" y="104.14"/>
 </segment>
 <segment>
@@
 <wire x1="40.64" y1="114.3" x2="35.56" y2="114.3" width="0.1524" layer="91"/>
 <label x="35.56" y="114.3" size="1.778" layer="95"/>
-<pinref part="S1" gate="1" pin="P"/>
-<wire x1="20.32" y1="106.68" x2="20.32" y2="114.3" width="0.1524" layer="91"/>
-<wire x1="20.32" y1="114.3" x2="30.48" y2="114.3" width="0.1524" layer="91"/>
-<wire x1="30.48" y1="114.3" x2="30.48" y2="106.68" width="0.1524" layer="91"/>
+<pinref part="S1" gate="1" pin="S1"/>
+<wire x1="30.48" y1="104.14" x2="30.48" y2="106.68" width="0.1524" layer="91"/>
 <junction x="30.48" y="106.68"/>
 </segment>
