File: Hardware/BEEP_0.1/TCS3103.brd (EAGLE design)
At the start: 28.2 x 30 mm, 15 parts, among them IC1 TCS3103

Commit message: Add branding ;) enhance PCBs finish Easy RGB Board add Texas Instruments libray from Element 14 add dxf import ulp for eagle add Script for easy eagle export to pdf for etching minor cleanup
Parts:
- removed U$2: (no value), holes:3,2
- added U$1: LOGO-COPPER4, Branding:COPPER4
Other:
- board text added: "TCS3103 v0.1.1"
Changed lines of the file:
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@@
 <layer number="43" name="vRestrict" color="2" fill="10" visible="yes" active="yes"/>
 <layer number="44" name="Drills" color="7" fill="1" visible="no" active="yes"/>
-<layer number="45" name="Holes" color="7" fill="1" visible="no" active="yes"/>
+<layer number="45" name="Holes" color="7" fill="1" visible="yes" active="yes"/>
 <layer number="46" name="Milling" color="3" fill="1" visible="no" active="yes"/>
 <layer number="47" name="Measures" color="7" fill="1" visible="no" active="yes"/>
-<layer number="48" name="Document" color="7" fill="1" visible="yes" active="yes"/>
-<layer number="49" name="Reference" color="7" fill="1" visible="yes" active="yes"/>
+<layer number="48" name="Document" color="7" fill="1" visible="no" active="yes"/>
+<layer number="49" name="Reference" color="7" fill="1" visible="no" active="yes"/>
 <layer number="51" name="tDocu" color="7" fill="1" visible="yes" active="yes"/>
 <layer number="52" name="bDocu" color="7" fill="1" visible="yes" active="yes"/>
@@
 <layer number="97" name="Info" color="7" fill="1" visible="no" active="no"/>
 <layer number="98" name="Guide" color="6" fill="1" visible="no" active="no"/>
+<layer number="100" name="tCName" color="7" fill="1" visible="yes" active="yes"/>
+<layer number="101" name="bCName" color="7" fill="1" visible="yes" active="yes"/>
 </layers>
 <board>
@@
 <text x="17.1" y="8" size="1.016" layer="26" rot="MR180" align="center-left">VOG</text>
 <text x="17.1" y="5.5" size="1.016" layer="26" rot="MR180" align="center-left">VOB</text>
+<text x="27.5" y="1.3" size="1.27" layer="100" rot="R90">TCS3103
+v0.1.1</text>
+<wire x1="21.5" y1="0" x2="21.5" y2="8.1" width="0.4064" layer="41"/>
+<wire x1="21.5" y1="8.1" x2="22.5" y2="9.1" width="0.4064" layer="41"/>
+<wire x1="22.5" y1="9.1" x2="28.2" y2="9.1" width="0.4064" layer="41"/>
+<wire x1="28.2" y1="9.1" x2="28.2" y2="0" width="0.4064" layer="41"/>
+<wire x1="28.2" y1="0" x2="21.5" y2="0" width="0.4064" layer="41"/>
 </plain>
 <attributes>
@@
 <attribute name="VALUE" x="9.96" y="21.57" size="1.016" layer="27" rot="R270"/>
 </element>
-<element name="U$2" library="holes" package="3,2" value="" x="24.1" y="4.1"/>
 <element name="U$3" library="holes" package="3,2" value="" x="4.2" y="4.1"/>
 <element name="U$4" library="holes" package="3,2" value="" x="24.1" y="25.7"/>
@@
 <attribute name="NAME" x="6.995" y="14.64" size="1.016" layer="25" align="center-left"/>
 </element>
+<element name="U$1" library="Branding" package="COPPER4" value="LOGO-COPPER4" x="23.9" y="1.4" rot="R90"/>
 </elements>
 <signals>
@@
 </signal>
 </signals>
-<errors>
-</errors>
 </board>
 </drawing>
+<compatibility>
+<note version="6.3" minversion="6.2.2" severity="warning">
+Since Version 6.2.2 text objects can contain more than one line,
+which will not be processed correctly with this version.
+</note>
+</compatibility>
 </eagle>
