File: Hardware/PCBs/BEEP_0.1/AIO.brd (EAGLE design)
At the start: 110 x 110 mm, 81 parts, among them IC1 ULN2803ASOP18, IC2 ULN2803ASOP18, IC3 74HC238D, IC4 74HC238D, U1 ATXMEGA64D3-AU, U2 TB6612FNG, X1 MICROMATCH-8, X10 MICROMATCH-10, X2 MICROMATCH-8, X3 MICROMATCH-8, X4 MICROMATCH-8, X5 MICROMATCH-8, X6 MICROMATCH-8, X7 MICROMATCH-8, X8 MICROMATCH-8, X9 MICROMATCH-4

Commit message: partly route the main beep board
Parts:
- removed R10, R11, R6, R7, R8, R9: (no value), rcl:R0603
- removed R38: 100R, rcl:R0603
- removed R39: 47K, rcl:R0603
- removed S1, S2: (no value), switch-omron:B3F-31XX
- removed U$4: DMN2075U, BEEP:SOT95P240X112-3N
- removed U1: ATXMEGA64D3-AU, atmel-xmega:TQFP-64A-64
- added U3: ATXMEGA64D3-AU, atmel-xmega:TQFP-64A-64
- moved LED10 76.8 mm to (46.2, 73.4), turned to 0 degrees
- moved LED9 76.0 mm to (48.2, 72.9), turned to 0 degrees
- moved R33 56.4 mm to (23.6, 46.9), turned to 90 degrees
- moved R32 56.4 mm to (23.6, 43.8), turned to 270 degrees
- moved R5 56.3 mm to (58.6, 65.8), turned to 0 degrees
- moved C4 51.1 mm to (27.4, 28.1), turned to 0 degrees
- moved R4 48.1 mm to (60.2, 61.4), turned to 0 degrees
- moved R30 47.3 mm to (50.4, 66.5), turned to 0 degrees
- moved R3 45.3 mm to (19.0, 67.6), turned to 180 degrees
- moved R35 45.0 mm to (27.6, 67.7), turned to 180 degrees
- moved C6 44.7 mm to (36.5, 45.8), turned to 0 degrees
- moved R31 44.0 mm to (54.0, 64.5), turned to 0 degrees
- moved C3 42.3 mm to (27.1, 31.9), turned to 0 degrees
- moved R2 41.6 mm to (19.0, 65.6), turned to 180 degrees
- moved U$3 40.2 mm to (22.2, 67.9), turned to 270 degrees
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Connections:
- removed net N$14: IC3.4, R7.2
- removed net N$15: IC3.5, R6.2
- removed net N$16: IC3.6, R8.1
- removed net N$17: IC4.4, R10.2
- removed net N$18: IC4.5, R9.2
- removed net N$22: S1.1, U$26.GPIO_23
- removed net N$25: S2.1, U$26.GPIO_22
- removed net N$35: IC4.6, R11.1
- removed net N$41: U$26.5V@1, U$26.5V@2, U$4.S
- removed net N$42: R38.2, R39.1, U$4.G
- removed net RPI_IKILL: R38.1, U1.26
- net +3V3: now also IC3.6, IC4.6, U3.15, U3.25, U3.35, U3.45, U3.53, U3.61; no longer R11.2, R8.2, U1.15, U1.25, U1.35, U1.45, U1.53, U1.61
- net +5V: now also U$26.5V@1, U$26.5V@2; no longer R39.2, U$4.D
- net ADISTANCE_0: now also U3.6; no longer U1.6
- net ADISTANCE_1: now also U3.7; no longer U1.7
- net ADISTANCE_2: now also U3.8; no longer U1.8
- net ADISTANCE_3: now also U3.9; no longer U1.9
- net ADISTANCE_4: now also U3.10; no longer U1.10
- net ADISTANCE_5: now also U3.11; no longer U1.11
- net ADISTANCE_6: now also U3.12; no longer U1.12
- net ADISTANCE_7: now also U3.13; no longer U1.13
- net BATT_VOLTAGE: now also U3.64; no longer U1.64
- net BATT_WARN_0: now also U3.1; no longer U1.1
- net BATT_WARN_1: now also U3.2; no longer U1.2
- net COLOR_DIODE_1: now also U3.31; no longer U1.41
- net COLOR_DIODE_2: now also U3.32; no longer U1.42
- net COLOR_FREQ_OUT: now also U3.26; no longer U1.38
- net COLOR_SENSOR_1: now also U3.33; no longer U1.43
- net COLOR_SENSOR_2: now also U3.27; no longer U1.39
- net COLOR_SENSOR_3: now also U3.30; no longer U1.40
- net COLOR_SENSOR_PWM_LED: now also U3.19; no longer U1.19
- net GND: now also IC3.4, IC3.5, IC4.4, IC4.5, U3.14, U3.24, U3.34, U3.44, U3.52, U3.60, U3.63; no longer R10.1, R6.1, R7.1, R9.1, S1.2, S2.2, U1.14, U1.24, U1.34, U1.44, U1.52, U1.60, U1.63
- net IR_LED_K4_OUT: now also IC2.13; no longer IC2.14
- net IR_LED_K5_OUT: now also IC2.12; no longer IC2.13
- net IR_LED_K6_OUT: now also IC2.11; no longer IC2.12
- net IR_LED_K7_OUT: now also IC2.14; no longer IC2.11
- net IR_LED_MK0: now also U3.48; no longer U1.48
- net IR_LED_MK1: now also U3.47; no longer U1.47
- net IR_LED_MK2: now also U3.46; no longer U1.46
- net LED_A0: now also U3.16; no longer U1.16
- net LED_A1: now also U3.17; no longer U1.17
- net LED_A2: now also U3.18; no longer U1.18
- net MOTOR_A_IN1: now also U3.41; no longer U1.30
- net MOTOR_A_IN2: now also U3.40; no longer U1.33
- net MOTOR_A_PWM: now also U3.39; no longer U1.20
- net MOTOR_B_IN1: now also U3.42; no longer U1.31
- net MOTOR_B_IN2: now also U3.43; no longer U1.32
- net MOTOR_B_PWM: now also U3.38; no longer U1.21
- net MOTOR_STBY: now also U3.22; no longer U1.22
- net N$4: now also U3.62; no longer U1.62
- net PDI_CLK: now also U3.57; no longer U1.57
- net PDI_DATA: now also U3.56; no longer U1.56
- net RGB_LED_MK0: now also U3.51; no longer U1.51
- net RGB_LED_MK1: now also U3.50; no longer U1.50
- net RGB_LED_MK2: now also U3.49; no longer U1.49
- net RPI_RX: now also U3.29; no longer U1.29
- net RPI_TX: now also U3.28; no longer U1.28
- net SCL: now also U3.37; no longer U1.37
- net SDA: now also U3.36; no longer U1.36
Routing:
- net LED_A0_OUT: track 0.00 -> 285.9 mm, vias 0 -> 7
- net LED_A2_OUT: track 0.00 -> 282.7 mm, vias 0 -> 8
- net LED_A1_OUT: track 20.3 -> 271.4 mm, vias 1 -> 8
- net +5V: track 47.5 -> 247.0 mm, vias 2 -> 10
- net LED_K4_OUT: track 0.00 -> 98.1 mm, vias 0 -> 1
- net LED_K5_OUT: track 0.00 -> 95.9 mm, vias 0 -> 2
- net ADISTANCE_2: track 0.00 -> 90.0 mm, vias 0 -> 1
- net ADISTANCE_3: track 0.00 -> 78.5 mm, vias 0 -> 4
- net ADISTANCE_1: track 0.00 -> 73.0 mm, vias 0 -> 2
- net SDA: track 0.00 -> 68.2 mm
- net SCL: track 0.00 -> 66.3 mm
- net PDI_CLK: track 62.1 -> 0.00 mm, vias 2 -> 0
- net IR_LED_K7_OUT: track 21.2 -> 81.3 mm, vias 0 -> 1
- net IR_LED_K6_OUT: track 46.5 -> 105.1 mm, vias 0 -> 3
- net GND: track 205.2 -> 260.7 mm, vias 2 -> 7
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
Commit message: continue routing
Parts:
- SV1: device con-ml:ML6 -> pinhead:2X03
- moved R34 11.6 mm to (58.3, 56.3), turned to 180 degrees
- moved R29 8.15 mm to (61.5, 59.0), turned to 270 degrees
- moved R31 7.06 mm to (48.9, 69.4), turned to 90 degrees
- moved R30 4.63 mm to (46.7, 69.3), turned to 90 degrees
- moved R5 4.22 mm to (58.2, 61.6)
- moved C10 3.36 mm to (36.9, 65.2), turned to 270 degrees
- moved LED10 2.75 mm to (48.9, 72.9)
- moved R4 2.55 mm to (59.4, 59.0), turned to 270 degrees
- moved U3 1.94 mm to (46.3, 55.9)
- moved C11 1.78 mm to (47.2, 42.6), turned to 270 degrees
- moved IC3 1.50 mm to (47.8, 35.9)
- moved LED9 1.50 mm to (46.7, 72.9)
- moved C7 1.40 mm to (50.3, 43.7)
- moved IC2 1.22 mm to (64.8, 27.6)
- moved C12 1.20 mm to (55.3, 42.7)
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Connections:
- net N$4: no longer U3.62
Routing:
- net GND: track 260.7 -> 411.7 mm, vias 7 -> 18
- net +3V3: track 118.1 -> 240.5 mm, vias 2 -> 6
- net ADISTANCE_4: track 34.2 -> 97.1 mm, vias 2 -> 5
- net LED_A0_OUT: track 285.9 -> 330.5 mm
- net LED_A2_OUT: track 282.7 -> 326.5 mm
- net ADISTANCE_5: track 34.2 -> 77.7 mm, vias 0 -> 3
- net LED_A1_OUT: track 271.4 -> 311.3 mm
- net +5V: track 247.0 -> 286.1 mm, vias 10 -> 12
- net MOTOR_STBY: track 3.32 -> 38.5 mm, vias 1 -> 2
- net RPI_TX: track 38.3 -> 63.7 mm
- net ADISTANCE_0: track 12.4 -> 37.6 mm, vias 0 -> 1
- net RPI_RX: track 35.7 -> 60.7 mm
- net PDI_CLK: track 0.00 -> 23.7 mm, vias 0 -> 3
- net PDI_DATA: track 0.00 -> 23.0 mm
- net ADISTANCE_6: track 32.3 -> 53.4 mm, vias 0 -> 4
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
Commit message: continue routing
Parts:
- moved IC3 1.80 mm to (49.6, 35.8)
Connections:
- net N$4: now also U3.62
Routing:
- net +3V3: track 240.5 -> 298.6 mm, vias 6 -> 10
- net GND: track 411.7 -> 451.0 mm, vias 18 -> 20
- net N$9: track 17.9 -> 15.4 mm
- net N$10: track 19.7 -> 17.3 mm
- net N$7: track 16.0 -> 13.7 mm
- net IR_LED_K1: track 12.9 -> 10.7 mm
- net N$6: track 14.4 -> 12.2 mm
- net IR_LED_K0: track 11.2 -> 9.52 mm
- net +5V: track 286.1 -> 287.8 mm
- net IR_LED_K4_OUT: track 81.8 -> 83.4 mm
- net N$12: track 20.8 -> 19.2 mm
- net LED_K6_OUT: track 91.8 -> 93.2 mm
- net LED_K7_OUT: track 93.4 -> 94.8 mm
- net LED_A2_OUT: track 326.5 -> 327.8 mm
- net LED_K5_OUT: track 97.8 -> 99.0 mm
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