File: Hardware/PCBs/BEEP_0.1/AIO.brd (EAGLE design)
At the start: 106.2 x 69.1 mm, 86 parts, among them IC1 ULN2803ASOP18, IC2 ULN2803ASOP18, IC3 74HC238SSOP, IC4 74HC238SSOP, IC5 TS34119SMD, U2 TB6612FNG, U3 ATXMEGA64D3-AU, X1 MICROMATCH-4, X10 MICROMATCH-10, X3 MICROMATCH-8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

Commit message: add critical DRC file continue routing
Parts:
- removed S2: (no value), switch-omron:B3F-10XX
- removed X14: (no value), con-amp:FSIDE-8
- added X2: (no value), con-amp:FSIDE-8
- moved R10 13.3 mm to (74.6, 27.9), turned to 0 degrees
- moved C14 12.4 mm to (74.6, 30.0), turned to 180 degrees
- moved X1 10.7 mm to (72.4, 9.00), turned to 0 degrees
- moved R9 7.40 mm to (68.9, 18.9), turned to 270 degrees
- moved IC5 6.89 mm to (75.8, 22.8), turned to 90 degrees
- moved C15 5.18 mm to (71.1, 18.9), turned to 90 degrees
- moved X3 2.00 mm to (83.9, 8.95)
- moved R8 1.00 mm to (43.5, 18.3)
- moved C9 0.82 mm to (58.0, 50.4)
- moved IC4 0.63 mm to (59.7, 44.2)
- moved R6 0.32 mm to (43.5, 20.4), turned to 0 degrees
- moved U$7 0.20 mm to (41.8, 25.5)
- moved C8 0.10 mm to (58.0, 57.2)
Connections:
- net +5V: now also X2.1; no longer X14.2
- net ADISTANCE_5: now also X2.2; no longer X14.3
- net AUDIO_DISABLE: now also U3.54
- net BATT_GND: now also U$5.D
- net GND: now also X2.3; no longer X14.4
- net IR_LED_K5_OUT: now also X2.4; no longer X14.5
- net LED_A0_OUT: now also X2.8
- net LED_A1_OUT: now also X2.7; no longer X14.8
- net LED_A2_OUT: now also X2.6; no longer X14.7
- net LED_K5_OUT: now also X2.5; no longer X14.6
Routing:
- net AUDIO_DISABLE: track 0.00 -> 52.2 mm, vias 0 -> 4
- net N$15: track 0.00 -> 30.4 mm, vias 0 -> 4
- net AUDIO_IN: track 0.00 -> 29.5 mm
- net SPEAKER_O2: track 0.00 -> 29.0 mm
- net +7V: track 171.0 -> 188.0 mm, vias 5 -> 7
- net SPEAKER_O1: track 0.00 -> 12.0 mm
- net N$36: track 0.00 -> 10.8 mm, vias 0 -> 2
- net IR_LED_K3_OUT: track 28.9 -> 39.1 mm
- net N$22: track 15.2 -> 23.9 mm
- net GND: track 610.7 -> 617.7 mm, vias 24 -> 25
- net IR_LED_K2_OUT: track 54.8 -> 60.9 mm
- net LED_K5_OUT: track 112.6 -> 106.6 mm
- net ADISTANCE_2: track 113.9 -> 108.6 mm
- net ADISTANCE_3: track 86.4 -> 90.8 mm
- net BATT_GND: track 17.8 -> 14.0 mm
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- added copper zone on layer 1, net GND
- added copper zone on layer 16, net GND
