File: Hardware/PCBs/BEEP_0.1/AIO.sch (EAGLE design)
At the start: 81 parts, among them IC1 ULN2803ASOP18, IC2 ULN2803ASOP18, IC3 74HC238D, IC4 74HC238D, U1 ATXMEGA64D3-AU, U2 TB6612FNG, X1 MICROMATCH-8, X10 MICROMATCH-10, X2 MICROMATCH-8, X3 MICROMATCH-8, X4 MICROMATCH-8, X5 MICROMATCH-8, X6 MICROMATCH-8, X7 MICROMATCH-8, X8 MICROMATCH-8, X9 MICROMATCH-4

Commit message: partly route the main beep board
Parts:
- removed R10, R11, R6, R7, R8, R9: (no value), rcl:R-EU_R0603
- removed R38: 100R, rcl:R-EU_R0603
- removed R39: 47K, rcl:R-EU_R0603
- removed S1, S2: (no value), switch-omron:31-XX
- removed U$4: DMN2075U, BEEP:DMN2075U
- renumbered U1 to U3
Connections:
- removed net N$14: IC3.G2A, R7.2
- removed net N$15: IC3.G2B, R6.2
- removed net N$16: IC3.G1, R8.1
- removed net N$17: IC4.G2A, R10.2
- removed net N$18: IC4.G2B, R9.2
- removed net N$22: S1.P, U$26.GPIO_23
- removed net N$25: S2.P, U$26.GPIO_22
- removed net N$35: IC4.G1, R11.1
- removed net N$41: U$26.5V, U$4.S
- removed net N$42: R38.2, R39.1, U$4.G
- removed net RPI_IKILL: R38.1, U3.PD0
- net +3V3: now also IC3.G1, IC4.G1; no longer R11.2, R8.2
- net +5V: now also U$26.5V; no longer R39.2, U$4.D
- net COLOR_DIODE_1: now also U3.PD5; no longer U3.PE5
- net COLOR_DIODE_2: now also U3.PD6; no longer U3.PE6
- net COLOR_FREQ_OUT: now also U3.PD0; no longer U3.PE2
- net COLOR_SENSOR_1: now also U3.PD7; no longer U3.PE7
- net COLOR_SENSOR_2: now also U3.PD1; no longer U3.PE3
- net COLOR_SENSOR_3: now also U3.PD4; no longer U3.PE4
- net GND: now also IC3.G2A, IC3.G2B, IC4.G2A, IC4.G2B; no longer R10.1, R6.1, R7.1, R9.1, S1.S, S2.S
- net IR_LED_K4_OUT: now also IC2.O6; no longer IC2.O5
- net IR_LED_K5_OUT: now also IC2.O7; no longer IC2.O6
- net IR_LED_K6_OUT: now also IC2.O8; no longer IC2.O7
- net IR_LED_K7_OUT: now also IC2.O5; no longer IC2.O8
- net MOTOR_A_IN1: now also U3.PE5; no longer U3.PD4
- net MOTOR_A_IN2: now also U3.PE4; no longer U3.PD7
- net MOTOR_A_PWM: now also U3.PE3; no longer U3.PC4
- net MOTOR_B_IN1: now also U3.PE6; no longer U3.PD5
- net MOTOR_B_IN2: now also U3.PE7; no longer U3.PD6
- net MOTOR_B_PWM: now also U3.PE2; no longer U3.PC5
Other:
- note removed: "Kill RPI on low batt"

Commit message: continue routing
Parts:
- SV1: device con-ml:ML6 -> pinhead:PINHD-2X3
Connections:
- net N$4: no longer U3.PA0
Changed lines of the file:
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@@
 <part name="+3V18" library="supply1" deviceset="+3V3" device=""/>
 <part name="+3V19" library="supply1" deviceset="+3V3" device=""/>
-<part name="SV1" library="con-ml" deviceset="ML6" device="" value="PDI"/>
+<part name="SV1" library="pinhead" deviceset="PINHD-2X3" device="" value="PDI"/>
 <part name="+3V20" library="supply1" deviceset="+3V3" device=""/>
 <part name="GND37" library="supply1" deviceset="GND" device=""/>
@@
 <instance part="+3V18" gate="G$1" x="215.9" y="187.96"/>
 <instance part="+3V19" gate="G$1" x="220.98" y="187.96"/>
-<instance part="SV1" gate="1" x="248.92" y="66.04" rot="R180"/>
+<instance part="SV1" gate="A" x="246.38" y="66.04"/>
 <instance part="+3V20" gate="G$1" x="264.16" y="78.74"/>
 <instance part="GND37" gate="1" x="261.62" y="58.42"/>
@@
 </segment>
 <segment>
-<pinref part="SV1" gate="1" pin="6"/>
+<pinref part="SV1" gate="A" pin="6"/>
 <pinref part="GND37" gate="1" pin="GND"/>
-<wire x1="256.54" y1="63.5" x2="261.62" y2="63.5" width="0.1524" layer="91"/>
+<wire x1="251.46" y1="63.5" x2="261.62" y2="63.5" width="0.1524" layer="91"/>
 <wire x1="261.62" y1="63.5" x2="261.62" y2="60.96" width="0.1524" layer="91"/>
 </segment>
@@
 </segment>
 <segment>
-<pinref part="SV1" gate="1" pin="2"/>
+<pinref part="SV1" gate="A" pin="2"/>
 <pinref part="+3V20" gate="G$1" pin="+3V3"/>
-<wire x1="256.54" y1="68.58" x2="264.16" y2="68.58" width="0.1524" layer="91"/>
+<wire x1="251.46" y1="68.58" x2="264.16" y2="68.58" width="0.1524" layer="91"/>
 <wire x1="264.16" y1="68.58" x2="264.16" y2="76.2" width="0.1524" layer="91"/>
 </segment>
@@
 <net name="PDI_DATA" class="0">
 <segment>
-<pinref part="SV1" gate="1" pin="1"/>
-<wire x1="241.3" y1="68.58" x2="233.68" y2="68.58" width="0.1524" layer="91"/>
+<pinref part="SV1" gate="A" pin="1"/>
+<wire x1="243.84" y1="68.58" x2="233.68" y2="68.58" width="0.1524" layer="91"/>
 <label x="233.68" y="68.58" size="1.27" layer="95" rot="R180" xref="yes"/>
 </segment>
@@
 <net name="PDI_CLK" class="0">
 <segment>
-<pinref part="SV1" gate="1" pin="5"/>
-<wire x1="241.3" y1="63.5" x2="233.68" y2="63.5" width="0.1524" layer="91"/>
+<pinref part="SV1" gate="A" pin="5"/>
+<wire x1="243.84" y1="63.5" x2="233.68" y2="63.5" width="0.1524" layer="91"/>
 <label x="233.68" y="63.5" size="1.27" layer="95" rot="R180" xref="yes"/>
 </segment>
@@
 <net name="N$4" class="0">
 <segment>
-<wire x1="129.54" y1="160.02" x2="175.26" y2="160.02" width="0.1524" layer="91"/>
 <pinref part="R4" gate="G$1" pin="1"/>
 <pinref part="R5" gate="G$1" pin="2"/>
-<junction x="175.26" y="160.02"/>
-<pinref part="U3" gate="G$1" pin="PA0"/>
-</segment>
-</net>
+</segment>
+</net>

Commit message: continue routing
Connections:
- net N$4: now also U3.PA0
Changed lines of the file:
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@@
 <pinref part="R4" gate="G$1" pin="1"/>
 <pinref part="R5" gate="G$1" pin="2"/>
+<pinref part="U3" gate="G$1" pin="PA0"/>
+<wire x1="129.54" y1="160.02" x2="175.26" y2="160.02" width="0.1524" layer="91"/>
+<junction x="175.26" y="160.02"/>
 </segment>
 </net>
