File: Hardware/PCBs/BEEP_0.1/AIO.sch (EAGLE design)
At the start: 84 parts, among them IC1 ULN2803ASOP18, IC2 ULN2803ASOP18, IC3 74HC238SSOP, IC4 74HC238SSOP, IC5 TS34119SMD, U2 TB6612FNG, U3 ATXMEGA64D3-AU, X1 MICROMATCH-4, X10 MICROMATCH-10, X3 MICROMATCH-8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

Commit message: add critical DRC file continue routing
Parts:
- removed S2: (no value), switch-omron:10-XX
- removed X14: (no value), con-amp:FSIDE-8
- added X2: (no value), con-amp:FSIDE-8
Connections:
- net +5V: now also X2-1.1; no longer X14-2.1
- net ADISTANCE_5: now also X2-2.1; no longer X14-3.1
- net AUDIO_DISABLE: now also U3.PF6
- net BATT_GND: now also U$5.D
- net GND: now also X2-3.1; no longer X14-4.1
- net IR_LED_K5_OUT: now also X2-4.1; no longer X14-5.1
- net LED_A0_OUT: now also X2-8.1
- net LED_A1_OUT: now also X2-7.1; no longer X14-8.1
- net LED_A2_OUT: now also X2-6.1; no longer X14-7.1
- net LED_K5_OUT: now also X2-5.1; no longer X14-6.1
Changed lines of the file:
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@@
 <part name="JP1" library="pinhead" deviceset="PINHD-1X5" device=""/>
 <part name="X11" library="con-amp" deviceset="FSIDE-8" device=""/>
-<part name="X14" library="con-amp" deviceset="FSIDE-8" device=""/>
 <part name="X15" library="con-amp" deviceset="FSIDE-8" device=""/>
 <part name="X16" library="con-amp" deviceset="FSIDE-8" device=""/>
@@
 <part name="GND42" library="supply1" deviceset="GND" device=""/>
 <part name="SUPPLY2" library="supply2" deviceset="+7V" device=""/>
-<part name="S2" library="switch-omron" deviceset="10-XX" device=""/>
 <part name="SUPPLY5" library="supply2" deviceset="+7V" device=""/>
 <part name="GND43" library="supply1" deviceset="GND" device=""/>
@@
 <part name="C15" library="rcl" deviceset="C-EU" device="C0603" value="1uF"/>
 <part name="X1" library="Con-amp-micromatch" deviceset="MICROMATCH-4" device=""/>
+<part name="X2" library="con-amp" deviceset="FSIDE-8" device=""/>
 </parts>
 <sheets>
@@
 <instance part="X11" gate="-7" x="175.26" y="345.44"/>
 <instance part="X11" gate="-8" x="175.26" y="342.9"/>
-<instance part="X14" gate="-1" x="228.6" y="363.22"/>
-<instance part="X14" gate="-2" x="228.6" y="360.68"/>
-<instance part="X14" gate="-3" x="228.6" y="358.14"/>
-<instance part="X14" gate="-4" x="228.6" y="355.6"/>
-<instance part="X14" gate="-5" x="228.6" y="353.06"/>
-<instance part="X14" gate="-6" x="228.6" y="350.52"/>
-<instance part="X14" gate="-7" x="228.6" y="347.98"/>
-<instance part="X14" gate="-8" x="228.6" y="345.44"/>
 <instance part="X15" gate="-1" x="175.26" y="330.2"/>
 <instance part="X15" gate="-2" x="175.26" y="327.66"/>
@@
 <instance part="GND42" gate="1" x="474.98" y="292.1"/>
 <instance part="SUPPLY2" gate="G$1" x="515.62" y="327.66"/>
-<instance part="S2" gate="1" x="541.02" y="307.34" rot="R270"/>
 <instance part="SUPPLY5" gate="G$1" x="408.94" y="327.66"/>
 <instance part="GND43" gate="1" x="408.94" y="299.72"/>
@@
 <instance part="X1" gate="-3" x="381" y="40.64"/>
 <instance part="X1" gate="-4" x="381" y="38.1"/>
+<instance part="X2" gate="-1" x="228.6" y="360.68"/>
+<instance part="X2" gate="-2" x="228.6" y="358.14"/>
+<instance part="X2" gate="-3" x="228.6" y="355.6"/>
+<instance part="X2" gate="-4" x="228.6" y="353.06"/>
+<instance part="X2" gate="-5" x="228.6" y="350.52"/>
+<instance part="X2" gate="-6" x="228.6" y="347.98"/>
+<instance part="X2" gate="-7" x="228.6" y="345.44"/>
+<instance part="X2" gate="-8" x="228.6" y="342.9"/>
 </instances>
 <busses>
@@
 <wire x1="198.12" y1="353.06" x2="198.12" y2="355.6" width="0.1524" layer="91"/>
 <wire x1="226.06" y1="355.6" x2="198.12" y2="355.6" width="0.1524" layer="91"/>
-<pinref part="X14" gate="-4" pin="1"/>
+<pinref part="X2" gate="-3" pin="1"/>
 </segment>
 <segment>
@@
 <wire x1="223.52" y1="360.68" x2="223.52" y2="363.22" width="0.1524" layer="91"/>
 <pinref part="P+15" gate="1" pin="+5V"/>
-<pinref part="X14" gate="-2" pin="1"/>
+<pinref part="X2" gate="-1" pin="1"/>
 </segment>
 <segment>
@@
 <net name="BATT_GND" class="0">
 <segment>
-<wire x1="370.84" y1="304.8" x2="373.38" y2="304.8" width="0.1524" layer="91"/>
-<label x="373.38" y="304.8" size="1.27" layer="95" xref="yes"/>
+<label x="378.46" y="304.8" size="1.27" layer="95" xref="yes"/>
+<pinref part="U$5" gate="G$1" pin="D"/>
+<wire x1="370.84" y1="304.8" x2="378.46" y2="304.8" width="0.1524" layer="91"/>
 </segment>
 <segment>
@@
 <wire x1="226.06" y1="350.52" x2="220.98" y2="350.52" width="0.1524" layer="91"/>
 <label x="220.98" y="350.52" size="1.27" layer="95" rot="R180" xref="yes"/>
-<pinref part="X14" gate="-6" pin="1"/>
+<pinref part="X2" gate="-5" pin="1"/>
 </segment>
 </net>
@@
 <wire x1="226.06" y1="347.98" x2="220.98" y2="347.98" width="0.1524" layer="91"/>
 <label x="220.98" y="347.98" size="1.27" layer="95" rot="R180" xref="yes"/>
-<pinref part="X14" gate="-7" pin="1"/>
+<pinref part="X2" gate="-6" pin="1"/>
 </segment>
 <segment>
@@
 <wire x1="226.06" y1="345.44" x2="220.98" y2="345.44" width="0.1524" layer="91"/>
 <label x="220.98" y="345.44" size="1.27" layer="95" rot="R180" xref="yes"/>
-<pinref part="X14" gate="-8" pin="1"/>
+<pinref part="X2" gate="-7" pin="1"/>
 </segment>
 <segment>
@@
 <wire x1="226.06" y1="342.9" x2="220.98" y2="342.9" width="0.1524" layer="91"/>
 <label x="220.98" y="342.9" size="1.27" layer="95" rot="R180" xref="yes"/>
+<pinref part="X2" gate="-8" pin="1"/>
 </segment>
 <segment>
@@
 <wire x1="226.06" y1="353.06" x2="220.98" y2="353.06" width="0.1524" layer="91"/>
 <label x="220.98" y="353.06" size="1.27" layer="95" rot="R180" xref="yes"/>
-<pinref part="X14" gate="-5" pin="1"/>
+<pinref part="X2" gate="-4" pin="1"/>
 </segment>
 <segment>
@@
 <wire x1="226.06" y1="358.14" x2="220.98" y2="358.14" width="0.1524" layer="91"/>
 <label x="220.98" y="358.14" size="1.27" layer="95" rot="R180" xref="yes"/>
-<pinref part="X14" gate="-3" pin="1"/>
+<pinref part="X2" gate="-2" pin="1"/>
 </segment>
 <segment>
@@
 <label x="373.38" y="91.44" size="1.27" layer="95" rot="R180" xref="yes"/>
 </segment>
-</net>
+<segment>
+<pinref part="U3" gate="G$1" pin="PF6"/>
+<wire x1="93.98" y1="76.2" x2="88.9" y2="76.2" width="0.1524" layer="91"/>
+<label x="88.9" y="76.2" size="1.27" layer="95" rot="R180" xref="yes"/>
+</segment>
+</net>
