File: Hardware/PCBs/BEEP_0.2/AIO.brd (EAGLE design)
At the start: 106.3 x 69.1 mm, 91 parts, among them IC1 74HC238SSOP, IC2 74HC238SSOP, IC3 ULN2803ASOP18, IC4 ULN2803ASOP18, IC5 ATXMEGA64D3-AU, IC6 GY-81, IC7 TB6612FNG, IC8 TS34119SMD, IC9 RASPBERRY-PI, Q1 DMN2075U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

Commit message: last? minor changes.
Parts:
- C13, C14: value (none) -> 10uF
- X11: value (none) -> line follow
- X12: value (none) -> motor
- X13: value (none) -> audio
- moved C3 0.10 mm to (49.0, 42.5)
- moved C5 0.10 mm to (51.1, 42.5)

Commit message: change value of cap in of off circuit continue case design
Parts:
- C17: value 1uF -> 4,7uF
Changed lines of the file:
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@@
 <element name="R24" library="resistor" package="M0805" value="100k" x="46.2" y="19.8" rot="R270"/>
 <element name="R30" library="resistor" package="M0805" value="10k" x="43" y="22" rot="R180"/>
-<element name="C17" library="resistor" package="M0805" value="1uF" x="46.2" y="15.8" rot="R270"/>
+<element name="C17" library="resistor" package="M0805" value="4,7uF" x="46.2" y="15.8" rot="R270"/>
 <element name="IC8" library="BEEP" package="SO08" value="TS34119SMD" x="76.6" y="22.8" rot="R90"/>
 <element name="R19" library="resistor" package="M0805" value="75k" x="68.6" y="18.8" rot="R270"/>
