File: Hardware/PCBs/BEEP_0.2/rgb_and_irdistance_side1.sch (EAGLE design)
At the start: 5 parts, among them IC1 HSDL-9100

Commit message: add more distance boards continue work on bottom pcb
Connections:
- net RGB_ANODE_1: now also U$1.6; no longer U$1.7
- net RGB_ANODE_2: now also U$1.7; no longer U$1.6
Changed lines of the file:
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@@
 </segment>
 <segment>
-<label x="218.44" y="81.28" size="1.27" layer="95" rot="R180" xref="yes"/>
-<pinref part="U$1" gate="G$1" pin="7"/>
-<wire x1="218.44" y1="81.28" x2="246.38" y2="81.28" width="0.1524" layer="91"/>
+<label x="218.44" y="83.82" size="1.27" layer="95" rot="R180" xref="yes"/>
+<pinref part="U$1" gate="G$1" pin="6"/>
+<wire x1="218.44" y1="83.82" x2="246.38" y2="83.82" width="0.1524" layer="91"/>
 </segment>
 </net>
@@
 </segment>
 <segment>
-<label x="218.44" y="83.82" size="1.27" layer="95" rot="R180" xref="yes"/>
-<pinref part="U$1" gate="G$1" pin="6"/>
-<wire x1="218.44" y1="83.82" x2="246.38" y2="83.82" width="0.1524" layer="91"/>
+<label x="218.44" y="81.28" size="1.27" layer="95" rot="R180" xref="yes"/>
+<pinref part="U$1" gate="G$1" pin="7"/>
+<wire x1="218.44" y1="81.28" x2="246.38" y2="81.28" width="0.1524" layer="91"/>
 </segment>
 </net>
