File: Hardware/PCBs/BEEP_0.2/bottom.sch (EAGLE design)
At the start: 58 parts, among them IC1 74HCT00D, Q1 DMN2075U, Q2 IRLML2244, Q5 IRLML2244, Q6 IRLML2244, Q8 IRLML2244, U1 LM239AMDREP, U2 ATTINY10-TSHR

Commit message: continue work on bottom pcb add simulation for attiny on/off
Parts:
- R9: value 10k -> 1k
Connections:
- removed net TINY_VCC: JP1.2
- net +3V3: now also C3.1, JP1.2; no longer R10.2
- net +5V: now also C2.1
- net +7V: now also R10.2
- net BATT_GND: no longer JP1.6
- net GND: now also C2.2, C3.2, JP1.6
Other:
- moved on the sheet: C2, C3
Changed lines of the file:
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@@
 <part name="GND21" library="supply1" deviceset="GND" device=""/>
 <part name="+3V15" library="supply1" deviceset="+3V3" device=""/>
-<part name="R9" library="rcl" deviceset="R-EU_" device="M0805" value="10k"/>
+<part name="R9" library="rcl" deviceset="R-EU_" device="M0805" value="1k"/>
 <part name="R10" library="rcl" deviceset="R-EU_" device="M0805" value="100k"/>
 <part name="R11" library="rcl" deviceset="R-EU_" device="M0805" value="1M"/>
@@
 <part name="C2" library="rcl" deviceset="C-EU" device="C0603"/>
 <part name="C3" library="rcl" deviceset="C-EU" device="C0603"/>
+<part name="SUPPLY2" library="supply2" deviceset="+7V" device=""/>
 <part name="+3V10" library="supply1" deviceset="+3V3" device=""/>
+<part name="GND17" library="supply1" deviceset="GND" device=""/>
+<part name="+3V11" library="supply1" deviceset="+3V3" device=""/>
+<part name="GND18" library="supply1" deviceset="GND" device=""/>
 </parts>
 <sheets>
@@
 <instance part="R32" gate="G$1" x="414.02" y="317.5" rot="MR0"/>
 <instance part="R33" gate="G$1" x="414.02" y="312.42" rot="MR0"/>
-<instance part="GND2" gate="1" x="60.96" y="66.04"/>
+<instance part="GND2" gate="1" x="66.04" y="66.04"/>
 <instance part="FRAME4" gate="G$1" x="0" y="193.04"/>
 <instance part="S1" gate="1" x="193.04" y="340.36" rot="R270"/>
@@
 <instance part="+3V9" gate="G$1" x="157.48" y="279.4"/>
 <instance part="C1" gate="G$1" x="96.52" y="297.18"/>
-<instance part="C2" gate="G$1" x="45.72" y="66.04"/>
-<instance part="C3" gate="G$1" x="408.94" y="297.18"/>
-<instance part="+3V10" gate="G$1" x="175.26" y="355.6"/>
+<instance part="C2" gate="G$1" x="48.26" y="66.04" rot="R90"/>
+<instance part="C3" gate="G$1" x="495.3" y="309.88"/>
+<instance part="SUPPLY2" gate="G$1" x="175.26" y="355.6"/>
+<instance part="+3V10" gate="G$1" x="495.3" y="317.5"/>
+<instance part="GND17" gate="1" x="495.3" y="299.72" rot="MR0"/>
+<instance part="+3V11" gate="G$1" x="134.62" y="243.84"/>
+<instance part="GND18" gate="1" x="134.62" y="226.06" rot="MR0"/>
 </instances>
 <busses>
@@
 <pinref part="GND2" gate="1" pin="GND"/>
 <wire x1="58.42" y1="71.12" x2="60.96" y2="71.12" width="0.1524" layer="91"/>
-<wire x1="60.96" y1="71.12" x2="60.96" y2="68.58" width="0.1524" layer="91"/>
+<wire x1="60.96" y1="71.12" x2="66.04" y2="71.12" width="0.1524" layer="91"/>
+<wire x1="66.04" y1="71.12" x2="66.04" y2="68.58" width="0.1524" layer="91"/>
+<pinref part="C2" gate="G$1" pin="2"/>
+<wire x1="53.34" y1="66.04" x2="60.96" y2="66.04" width="0.1524" layer="91"/>
+<wire x1="60.96" y1="66.04" x2="60.96" y2="71.12" width="0.1524" layer="91"/>
+<junction x="60.96" y="71.12"/>
 </segment>
 <segment>
@@
 <junction x="96.52" y="292.1"/>
 </segment>
+<segment>
+<pinref part="GND17" gate="1" pin="GND"/>
+<pinref part="C3" gate="G$1" pin="2"/>
+<wire x1="495.3" y1="302.26" x2="495.3" y2="304.8" width="0.1524" layer="91"/>
+</segment>
+<segment>
+<pinref part="JP1" gate="A" pin="6"/>
+<wire x1="124.46" y1="231.14" x2="134.62" y2="231.14" width="0.1524" layer="91"/>
+<pinref part="GND18" gate="1" pin="GND"/>
+<wire x1="134.62" y1="231.14" x2="134.62" y2="228.6" width="0.1524" layer="91"/>
+</segment>
 </net>
 <net name="+5V" class="0">
@@
 <pinref part="IC1" gate="P" pin="VCC"/>
 <pinref part="P+7" gate="1" pin="+5V"/>
-<wire x1="43.18" y1="71.12" x2="38.1" y2="71.12" width="0.1524" layer="91"/>
+<wire x1="43.18" y1="71.12" x2="40.64" y2="71.12" width="0.1524" layer="91"/>
+<wire x1="40.64" y1="71.12" x2="38.1" y2="71.12" width="0.1524" layer="91"/>
 <wire x1="38.1" y1="71.12" x2="38.1" y2="76.2" width="0.1524" layer="91"/>
+<pinref part="C2" gate="G$1" pin="1"/>
+<wire x1="45.72" y1="66.04" x2="40.64" y2="66.04" width="0.1524" layer="91"/>
+<wire x1="40.64" y1="66.04" x2="40.64" y2="71.12" width="0.1524" layer="91"/>
+<junction x="40.64" y="71.12"/>
 </segment>
 <segment>
@@
 </segment>
 <segment>
-<pinref part="R10" gate="G$1" pin="2"/>
 <pinref part="+3V10" gate="G$1" pin="+3V3"/>
-<wire x1="175.26" y1="350.52" x2="175.26" y2="353.06" width="0.1524" layer="91"/>
+<pinref part="C3" gate="G$1" pin="1"/>
+<wire x1="495.3" y1="314.96" x2="495.3" y2="312.42" width="0.1524" layer="91"/>
+</segment>
+<segment>
+<pinref part="JP1" gate="A" pin="2"/>
+<wire x1="124.46" y1="236.22" x2="134.62" y2="236.22" width="0.1524" layer="91"/>
+<pinref part="+3V11" gate="G$1" pin="+3V3"/>
+<wire x1="134.62" y1="236.22" x2="134.62" y2="241.3" width="0.1524" layer="91"/>
 </segment>
 </net>
@@
 <junction x="193.04" y="241.3"/>
 </segment>
+<segment>
+<pinref part="R10" gate="G$1" pin="2"/>
+<wire x1="175.26" y1="350.52" x2="175.26" y2="353.06" width="0.1524" layer="91"/>
+<pinref part="SUPPLY2" gate="G$1" pin="+7V"/>
+</segment>
 </net>
 <net name="BATT_GND" class="0">
-<segment>
-<pinref part="JP1" gate="A" pin="6"/>
-<wire x1="124.46" y1="231.14" x2="132.08" y2="231.14" width="0.1524" layer="91"/>
-<label x="132.08" y="231.14" size="1.27" layer="95" xref="yes"/>
-</segment>
 <segment>
 <pinref part="JP4" gate="A" pin="2"/>
@@
 </segment>
 </net>
-<net name="TINY_VCC" class="0">
-<segment>
-<pinref part="JP1" gate="A" pin="2"/>
-<wire x1="124.46" y1="236.22" x2="132.08" y2="236.22" width="0.1524" layer="91"/>
-<label x="132.08" y="236.22" size="1.27" layer="95" xref="yes"/>
-</segment>
-</net>

Commit message: minor pcb changes
Parts:
- C1: value (none) -> 100n
Other:
- moved on the sheet: JP1
Changed lines of the file:
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@@
 <part name="+3V8" library="supply1" deviceset="+3V3" device=""/>
 <part name="+3V9" library="supply1" deviceset="+3V3" device=""/>
-<part name="C1" library="rcl" deviceset="C-EU" device="C0603"/>
+<part name="C1" library="rcl" deviceset="C-EU" device="C0603" value="100n"/>
 <part name="C2" library="rcl" deviceset="C-EU" device="C0603"/>
 <part name="C3" library="rcl" deviceset="C-EU" device="C0603"/>
@@
 <instance part="GND23" gate="1" x="147.32" y="246.38" rot="MR0"/>
 <instance part="SUPPLY1" gate="G$1" x="147.32" y="281.94"/>
-<instance part="JP1" gate="A" x="119.38" y="233.68"/>
+<instance part="JP1" gate="A" x="121.92" y="228.6"/>
 <instance part="U2" gate="A" x="119.38" y="297.18"/>
 <instance part="R36" gate="G$1" x="157.48" y="269.24" rot="MR90"/>
@@
 <instance part="+3V10" gate="G$1" x="495.3" y="317.5"/>
 <instance part="GND17" gate="1" x="495.3" y="299.72" rot="MR0"/>
-<instance part="+3V11" gate="G$1" x="134.62" y="243.84"/>
-<instance part="GND18" gate="1" x="134.62" y="226.06" rot="MR0"/>
+<instance part="+3V11" gate="G$1" x="137.16" y="238.76"/>
+<instance part="GND18" gate="1" x="137.16" y="220.98" rot="MR0"/>
 </instances>
 <busses>
@@
 <segment>
 <pinref part="JP1" gate="A" pin="6"/>
-<wire x1="124.46" y1="231.14" x2="134.62" y2="231.14" width="0.1524" layer="91"/>
+<wire x1="127" y1="226.06" x2="137.16" y2="226.06" width="0.1524" layer="91"/>
 <pinref part="GND18" gate="1" pin="GND"/>
-<wire x1="134.62" y1="231.14" x2="134.62" y2="228.6" width="0.1524" layer="91"/>
+<wire x1="137.16" y1="226.06" x2="137.16" y2="223.52" width="0.1524" layer="91"/>
 </segment>
 </net>
@@
 <segment>
 <pinref part="JP1" gate="A" pin="2"/>
-<wire x1="124.46" y1="236.22" x2="134.62" y2="236.22" width="0.1524" layer="91"/>
+<wire x1="127" y1="231.14" x2="137.16" y2="231.14" width="0.1524" layer="91"/>
 <pinref part="+3V11" gate="G$1" pin="+3V3"/>
-<wire x1="134.62" y1="236.22" x2="134.62" y2="241.3" width="0.1524" layer="91"/>
+<wire x1="137.16" y1="231.14" x2="137.16" y2="236.22" width="0.1524" layer="91"/>
 </segment>
 </net>
@@
 <segment>
 <pinref part="JP1" gate="A" pin="1"/>
-<wire x1="116.84" y1="236.22" x2="109.22" y2="236.22" width="0.1524" layer="91"/>
-<label x="109.22" y="236.22" size="1.27" layer="95" rot="R180" xref="yes"/>
+<wire x1="119.38" y1="231.14" x2="111.76" y2="231.14" width="0.1524" layer="91"/>
+<label x="111.76" y="231.14" size="1.27" layer="95" rot="R180" xref="yes"/>
 </segment>
 </net>
@@
 <segment>
 <pinref part="JP1" gate="A" pin="3"/>
-<wire x1="116.84" y1="233.68" x2="109.22" y2="233.68" width="0.1524" layer="91"/>
-<label x="109.22" y="233.68" size="1.27" layer="95" rot="R180" xref="yes"/>
+<wire x1="119.38" y1="228.6" x2="111.76" y2="228.6" width="0.1524" layer="91"/>
+<label x="111.76" y="228.6" size="1.27" layer="95" rot="R180" xref="yes"/>
 </segment>
 </net>
@@
 <segment>
 <pinref part="JP1" gate="A" pin="5"/>
-<wire x1="116.84" y1="231.14" x2="109.22" y2="231.14" width="0.1524" layer="91"/>
-<label x="109.22" y="231.14" size="1.27" layer="95" rot="R180" xref="yes"/>
-</segment>
-<segment>
+<wire x1="119.38" y1="226.06" x2="111.76" y2="226.06" width="0.1524" layer="91"/>
+<label x="111.76" y="226.06" size="1.27" layer="95" rot="R180" xref="yes"/>
+</segment>
+<segment>
