File: Hardware/PCBs/eval_boards/tiny10.sch (EAGLE design)
At the start: 62 parts, among them IC1 74HCT00D, Q2 IRLML2244, Q3 IRLML2244, Q5 IRLML2244, Q6 IRLML2244, Q8 IRLML2244, U1 LM239AMDREP, U2 ATTINY10-TSHR

Commit message: the forgotten commit ;)
* enhance bottom, rgb sensor pcb
* create attiny and lm239 eval boards
* bug fix for the pdf export scripts
* correct attiny soft power switch simulation
* add experimental color sensor code
* add rgb color look up table
* correct motor roations
* various other (this is the forgetten commit)
Parts:
- removed C2: 100n, rcl:C-EUC0603
- removed C3: (no value), rcl:C-EUC0603
- removed D1, D2, D3, D4: CNY70, BEEP:CNY70
- removed D5, D6: BAS40, diode:BAS40
- removed IC1: 74HCT00D, 74xx-eu:74HCT00D
- removed JP4: (no value), pinhead:PINHD-1X3
- removed JP5: (no value), pinhead:PINHD-1X9
- removed LED1: (no value), led:LEDCHIP-LED0603
- removed Q2, Q3, Q5, Q6, Q8: IRLML2244, BEEP:IRLML2244
- removed R1, R2, R3, R4: 10k, rcl:R-EU_R0603
- removed R11: 100R, rcl:R-EU_M0805
- removed R12: 330R, rcl:R-EU_R0805
- removed R13, R15, R17, R19, R25, R37, R41: 10k, rcl:R-EU_M0805
- removed R14, R16, R18: 330R, rcl:R-EU_M0805
- removed R20, R21, R22, R23: 4.7k, rcl:R-EU_M0805
- removed R24: 5.6k, rcl:R-EU_M0805
- removed R26, R27, R28, R29, R39: 100k, rcl:R-EU_M0805
- removed R30, R31, R32, R33: 1M, rcl:R-EU_M0805
- removed R34, R35: (no value), rcl:R-EU_M0805
- removed R40: 1k, rcl:R-EU_M0805
- removed R5, R6, R7: 22R, rcl:R-EU_M0805
- removed R8: 0, rcl:R-EU_M0805
- removed S1: (no value), switch-omron:10-XX
- removed T1: (no value), transistor:-NPN-SOT23-EBC
- removed U1: LM239AMDREP, Texas Instruments_By_element14_Batch_1:LM239AMDREP
- removed X1: (no value), con-ftop-orientation-hole:FTOP-10
- added JP1: (no value), pinhead:PINHD-2X3
- added R36: (no value), rcl:R-EU_M0805
- JP2: device pinhead:PINHD-1X5 -> pinhead:PINHD-1X3
- JP3: device pinhead:PINHD-2X4 -> pinhead:PINHD-1X3
Connections:
- removed net !OFF!: R40.2, R41.2, T1.B, U2.PB0
- removed net +5V: C2.1, D1.LED_A, D2.LED_A, D3.LED_A, D4.LED_A, IC1P.VCC, JP2.5, Q2.S, Q5.S, Q6.S, Q8.S
- removed net BATT: JP4.2, Q3.S, R37.2
- removed net COLOR_DIODE_1: JP5.5, X1-4.1
- removed net COLOR_DIODE_2: JP5.4, X1-3.1
- removed net COLOR_FREQ_OUT: JP5.6, X1-7.1
- removed net COLOR_SENSOR_1: JP5.9, X1-2.1
- removed net COLOR_SENSOR_2: JP5.8, X1-6.1
- removed net COLOR_SENSOR_3: JP5.7, X1-5.1
- removed net COLOR_SENSOR_PWM_LED: JP5.3, X1-9.1
- removed net ENC_L1: JP2.1, R20.1, R30.1, U1.1OUT
- removed net ENC_L1_RAW: D1.T_E, R13.2, R26.2
- removed net ENC_L2: JP2.2, R21.1, R31.1, U1.2OUT
- removed net ENC_L2_RAW: D2.T_E, R15.2, R27.2
- removed net ENC_R1: JP2.3, R22.1, R32.1, U1.OUT3
- removed net ENC_R1_RAW: D3.T_E, R17.2, R28.2
- removed net ENC_R2: JP2.4, R23.1, R33.1, U1.OUT4
- removed net ENC_R2_RAW: D4.T_E, R19.2, R29.2
- removed net N$1: IC1A.O, Q5.G
- removed net N$13: Q8.D, R4.2, R8.1
- removed net N$14: Q6.D, R3.2, R7.1
- removed net N$15: Q2.D, R2.2, R6.1
- removed net N$2: IC1B.O, Q2.G
- removed net N$3: Q5.D, R1.2, R5.1
- removed net N$4: IC1C.O, Q6.G
- removed net N$43: D1.LED_C, R12.2
- removed net N$44: R26.1, R30.2, U1.1IN+
- removed net N$45: R27.1, R31.2, U1.2IN+
- removed net N$46: D2.LED_C, R14.2
- removed net N$47: R28.1, R32.2, U1.3IN+
- removed net N$48: D3.LED_C, R16.2
- removed net N$49: R29.1, R33.2, U1.4IN+
- removed net N$5: IC1D.O, Q8.G
- removed net N$50: D4.LED_C, R18.2
- removed net N$6: LED1.C, R11.2
- removed net N$8: D5.A, Q3.G, R37.1, T1.C
- removed net N$9: D5.C, D6.C, S1.S, S1.S1
- removed net PWM_IN1: IC1A.I0, IC1A.I1, JP3.2
- removed net PWM_IN2: IC1B.I0, IC1B.I1, JP3.4
- removed net PWM_IN3: IC1C.I0, IC1C.I1, JP3.6
- removed net PWM_IN4: IC1D.I0, IC1D.I1, JP3.8
- removed net PWM_OUT1: JP3.1, R5.2
- removed net PWM_OUT2: JP3.3, R6.2
- removed net PWM_OUT3: JP3.5, R7.2
- removed net PWM_OUT4: JP3.7, R8.2
- removed net RESET: R34.2, R35.1, U2.PB3
- removed net SENS: D6.A, R39.1, U2.PB2
- removed net SWITCHED_BATT: JP4.1, Q3.D, R35.2, R41.1
- removed net U_REF: R24.1, R25.2, U1.1IN-, U1.2IN-, U1.3IN-, U1.4IN-
- new net PB0/TPIDATA: JP1.1, JP2.1, U2.PB0
- new net PB2/SOFT_OFF: JP3.1, U2.PB2
- new net PB3/RESET: JP1.5, JP3.3, R36.1, U2.PB3
- net +3V3: now also JP1.2, JP3.2, R36.2; no longer C3.1, D1.T_C, D2.T_C, D3.T_C, D4.T_C, JP5.2, R20.2, R21.2, R22.2, R23.2, R24.2, R39.2, U1.VCC, X1-10.1
- net GND: now also JP1.6, JP2.2; no longer C2.2, C3.2, IC1P.GND, JP4.3, JP5.1, R1.1, R11.1, R12.1, R13.1, R14.1, R15.1, R16.1, R17.1, R18.1, R19.1, R2.1, R25.1, R3.1, R34.1, R4.1, R40.1, S1.P, S1.P1, T1.E, U1.GND, X1-8.1
- net PB1/TPICLK: now also JP1.3, JP2.3; no longer LED1.A
Other:
- moved on the sheet: C1, U2
